File: Projects/Client Name/Project Name/Design/rev01/rev01_1/DF_ESC_rev01_1/MOSFET DRIVER.kicad_sch (KiCad schematic)
At the start: 0 parts

Commit message: Update3
-MOSFET DRIVER circuit
Parts:
- added C18: 6n8, symbol Device:C
- added C19: 120p, symbol Device:C
- added C20, C21, C22, C23, C24, C25: 2U2, symbol Device:C
- added C26, C27, C28: 10u, symbol Device:C
- added R10: 205K, symbol Device:R
- added R11: 16K2, symbol Device:R
- added R12: 18K, symbol Device:R
- added R13: 3K3, symbol Device:R
- added R14: 10K, symbol Device:R
- added U2: DRV8302_DCA_56, DCA56_6P35X3P61, symbol DRV8302:DRV8302_DCA_56
Connections:
- new net: C18.1, R11.2
- new net: C19.1, R11.1, U2.2 (COMP)
- new net: R12.2, R13.1, U2.3 (VSENSE)
- new net: C22.1, C23.1, U2.13 (GVDD)
- new net: R10.1, U2.1 (RT_CLK)
- new net: C26.1, C27.1, C28.1, U2.29 (PVDD1)
- new net: R14.2, U2.7 (DTC)
- new net: C24.1, U2.14 (CP1)
- new net: C24.2, U2.15 (CP2)
- new net: C25.1, U2.27 (AVDD)
- new net +3V3: U2.24 (REF), U2.9 (M_OC)
- new net +5V: R12.1
- new net BR_SO1: U2.25 (SO1)
- new net BR_SO2: U2.26 (SO2)
- new net DC_CAL: U2.12 (DC_CAL)
- new net DVDD: C20.1, C21.1, U2.11 (OC_ADJ), U2.23 (DVDD)
- new net EN_GATE: U2.16 (EN_GATE)
- new net FAULT: U2.6 (*FAULT)
- new net GND: C18.2, C19.2, C20.2, C21.2, C22.2, C23.2, C25.2, C26.2, C27.2, C28.2, R10.2, R13.2, R14.1, U2.10 (GAIN), U2.28 (AGND), U2.8 (M_PWM)
- new net H1: U2.17 (INH_A)
- new net H2: U2.19 (INH_B)
- new net H3: U2.21 (INH_C)
- new net L1: U2.18 (INL_A)
- new net L2: U2.20 (INL_B)
- new net L3: U2.22 (INL_C)
- no-connect marks 0 -> 2
Other:
- note added: "BULK CAPACITANCE KEEP AS CLOSE AS POSSIBLE TO THE IC AND TO THE DRIVER INPUT LOOP"
