File: Projects/Client Name/Project Name/Design/rev01/rev01_1/DF_ESC_rev01_1/MUS.kicad_sch (KiCad schematic)
At the start: 0 parts

Commit message: Update3
-Microcontroller schematic design done
Parts:
- added 0R, R1, R2: R, symbol Device:R
- added C1, C12, C16, C17, C2, C4, C5, C6, C7, C8, C9: 100n, symbol Device:C
- added C10, C11: 2u2, symbol Device:C
- added C13: 1u, symbol Device:C
- added C14: 10p, symbol Device:C
- added C15: C, symbol Device:C
- added C3: 10u, symbol Device:C
- added D1: LED, symbol Device:LED
- added D2: LED_G, symbol Device:LED
- added D3: LED_R, symbol Device:LED
- added FB1: FerriteBead, symbol Device:FerriteBead
- added J1: Conn_01x06, symbol Connector_Generic:Conn_01x06
- added J2: Conn_01x03, symbol Connector_Generic:Conn_01x03
- added J3: Conn_01x08, symbol Connector_Generic:Conn_01x08
- added R3, R7, R9: 2K2, symbol Device:R
- added R4, R5, R6: 1K, symbol Device:R
- added R8: 39K, symbol Device:R
- added SW1: SW_DIP_x01, symbol Switch:SW_DIP_x01
- added TH1: 10K, symbol Device:Thermistor_NTC
- added U1: STM32F405RGTx, Package_QFP:LQFP-64_10x10mm_P0.5mm, symbol MCU_ST_STM32F4:STM32F405RGTx
- added Y1: Crystal, symbol Device:Crystal
Connections:
- new net: D1.2 (A), R4.2
- new net: D2.2 (A), R5.2
- new net: C15.2, R2.1, Y1.2
- new net: C12.1, C13.1, FB1.1, U1.13 (VDDA)
- new net: J2.3 (Pin_3), R3.2
- new net: R2.2, U1.5 (PH0)
- new net: D3.2 (A), R6.2
- new net: C10.1, U1.31 (VCAP_1)
- new net: 0R.1, C14.2, Y1.1
- new net: 0R.2, U1.6 (PH1)
- new net: C11.1, U1.47 (VCAP_2)
- new net: R1.2, U1.60 (BOOT0)
- new net +3V3: C16.1, C2.1, C3.1, C4.1, C5.1, C6.1, C7.1, C8.1, FB1.2, J1.1 (Pin_1), J3.2 (Pin_2), R1.1, R4.1, TH1.1, U1.1 (VBAT), U1.19 (VDD), U1.32 (VDD), U1.48 (VDD), U1.64 (VDD)
- new net +5V: J2.1 (Pin_1), J3.1 (Pin_1)
- new net +VDC: R8.1
- new net ADC_TEMP: R7.2, TH1.2, U1.17 (PA3)
- new net AN_IN: C17.2, R8.2, R9.1, U1.10 (PC2)
- new net BR_SO1: U1.27 (PB1)
- new net BR_SO2: U1.26 (PB0)
- new net CAN_RX: U1.61 (PB8)
- new net CAN_TX: U1.62 (PB9)
- new net DC_CAL: U1.33 (PB12)
- new net EN_GATE: U1.51 (PC10)
- new net FAULT: U1.53 (PC12)
- new net GND: C1.2, C10.2, C11.2, C12.2, C13.2, C14.1, C15.1, C16.2, C17.1, C2.2, C3.2, C4.2, C5.2, C6.2, C7.2, C8.2, C9.2, D1.1 (K), D2.1 (K), D3.1 (K), J1.3 (Pin_3), J2.2 (Pin_2), J3.3 (Pin_3), J3.8 (Pin_8), R7.1, R9.2, SW1.1, U1.12 (VSSA), U1.18 (VSS), U1.63 (VSS)
- new net H1: U1.43 (PA10)
- new net H2: U1.42 (PA9)
- new net H3: U1.41 (PA8)
- new net HALL_1: U1.58 (PB6)
- new net HALL_2: U1.59 (PB7)
- new net HALL_3: U1.52 (PC11)
- new net L1: U1.36 (PB15)
- new net L2: U1.35 (PB14)
- new net L3: U1.34 (PB13)
- new net LED_GREEN: R5.1, U1.24 (PC4)
- new net LED_RED: R6.1, U1.25 (PC5)
- new net MISO_ADC_EXT2: J3.7 (Pin_7), U1.22 (PA6)
- new net NRST: C9.1, J1.5 (Pin_5), SW1.2, U1.7 (NRST)
- new net RX_SCL_MOSI: J3.6 (Pin_6), U1.23 (PA7), U1.29 (PB10), U1.38 (PC7)
- new net SCK_ADC_EXT: J3.4 (Pin_4), U1.21 (PA5)
- new net SENS1: U1.16 (PA2)
- new net SENS2: U1.15 (PA1)
- new net SENS3: U1.14 (PA0)
- new net SERVO: C1.1, R3.1, U1.57 (PB5)
- new net SWCLK: J1.2 (Pin_2), U1.49 (PA14)
- new net SWDIO: J1.4 (Pin_4), U1.46 (PA13)
- new net TEMP_MOTOR: U1.8 (PC0)
- new net TX_SDA_NSS: J3.5 (Pin_5), U1.20 (PA4), U1.30 (PB11), U1.37 (PC6)
- new net USB_DM: U1.44 (PA11)
- new net USM_DP: U1.45 (PA12)
- no-connect marks 0 -> 13
Other:
- note added: "100nF Decoupling capacitors. Place one as close as possible to each pin."
- note added: "Boot mode table 7"
- note added: "COMMUNICATION"
- note added: "NRST: Internally Pulled-up"
- note added: "NTC THERMISTOR"
- note added: "Programming/Debug"
- note added: "SERVO"
- note added: "SUITABLE WITH 100R IF USED AS SERO OUTPUT"
- note added: "VOLTAGE_DIVIDER"
- note added: "WHEN: VDC = 60V => AN_IN = 3V204"
